File: Supercap.kicad_pcb (KiCad board)
At the start: 4 copper layers, 151.8 x 70 mm, 73 parts, among them IC1 NCP5109ADR2G, IC2 NCP5109ADR2G, J1 XT30, J2 XT30, J2-J1 Conn_01x10, J3 Conn_01x01, J3-J1 Conn_01x10, J4 Conn_01x01, P7803B-1000R1 P7803B-1000, P7812B-1000R1 490-P7812B-1000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

Commit message: small things, trevor checked, awaiting heavenly mandated egan
Parts:
- moved U6 16.3 mm to (247.8, 62.3)
- moved C_{smooth}3 1.38 mm to (172.2, 80.2), turned to -90 degrees
Routing:
- net GNDPWR: vias 50 -> 57
- net /Control/+3V3: vias 11 -> 12
Changed lines of the file:
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@@
 	(footprint "MSPM0:ti_LP_MSPM0G3507"
 		(layer "F.Cu")
-		(at 243.93 46.53 -90)
+		(at 247.83 62.33 -90)
 		(property "Reference" "U6"
 			(at -22.86 -45.72 90)
@@
 			(layer "Cmts.User")
 			(pts
-				(xy 246.47 54.15) (xy 297.27 54.15)
+				(xy 250.37 69.95) (xy 301.17 69.95)
 			)
 			(height 5.08)
@@
 			)
 			(gr_text "2.000"
-				(at 271.87 58.13 0)
+				(at 275.77 73.93 0)
 				(layer "Cmts.User")
 				(effects
@@
 			(layer "Cmts.User")
 			(pts
-				(xy 276.95 18.59) (xy 276.95 74.47)
+				(xy 280.85 34.39) (xy 280.85 90.27)
 			)
 			(height -2.54)
@@
 			)
 			(gr_text "2.200"
-				(at 278.39 46.53 90)
+				(at 282.29 62.33 90)
 				(layer "Cmts.User")
 				(effects
@@
 			(layer "Cmts.User")
 			(pts
-				(xy 223.61 59.23) (xy 193.13 59.23)
+				(xy 227.51 75.03) (xy 197.03 75.03)
 			)
 			(height -2.54)
@@
 			)
 			(gr_text "1.200"
-				(at 208.37 60.67 0)
+				(at 212.27 76.47 0)
 				(layer "Cmts.User")
 				(effects
@@
 			(layer "Cmts.User")
 			(pts
-				(xy 297.27 33.83) (xy 193.13 33.83)
+				(xy 301.17 49.63) (xy 197.03 49.63)
 			)
 			(height -5.08)
@@
 			)
 			(gr_text "4.100"
-				(at 245.2 37.81 0)
+				(at 249.1 53.61 0)
 				(layer "Cmts.User")
 				(effects
@@
 	(footprint "Capacitor_SMD:C_0603_1608Metric_Pad1.08x0.95mm_HandSolder"
 		(layer "F.Cu")
-		(at 171.2125 81.16)
+		(at 172.17 80.1625 -90)
 		(descr "Capacitor SMD 0603 (1608 Metric), square (rectangular) end terminal, IPC_7351 nominal with elongated pad for handsoldering. (Body size source: IPC-SM-782 page 76, https://www.pcb-3d.com/wordpress/wp-content/uploads/ipc-sm-782a_amendment_1_and_2.pdf), generated with kicad-footprint-generator")
 		(tags "capacitor handsolder")
 		(property "Reference" "C_{smooth}3"
-			(at 0 -1.43 0)
+			(at 0 -1.43 90)
 			(layer "F.SilkS")
 			(effects
@@
 		)
 		(property "Value" "4.7u"
-			(at 0 1.43 0)
+			(at 0 1.43 90)
 			(layer "F.Fab")
 			(effects
@@
 		)
 		(property "Datasheet" "https://weblib.samsungsem.com/mlcc/mlcc-ec-data-sheet.do?partNumber=CL10A475KO8NNN"
-			(at 0 0 0)
+			(at 0 0 270)
 			(unlocked yes)
 			(layer "F.Fab")
@@
 		)
 		(property "Description" "Unpolarized capacitor"
-			(at 0 0 0)
+			(at 0 0 270)
 			(unlocked yes)
 			(layer "F.Fab")
@@
 		)
 		(property "Mouser#" ""
-			(at 0 0 0)
+			(at 0 0 270)
 			(unlocked yes)
 			(layer "F.Fab")
@@
 		)
 		(property "Manufacturer_Part_Number" "CL10A475KO8NNNC"
-			(at 0 0 0)
+			(at 0 0 270)
 			(unlocked yes)
 			(layer "F.Fab")
@@
 		)
 		(property "Mouser Part Number" "187-CL10A475KO8NNNC"
-			(at 0 0 0)
+			(at 0 0 270)
 			(unlocked yes)
 			(layer "F.Fab")
@@
 		(attr smd)
 		(fp_line
-			(start -0.146267 -0.51)
-			(end 0.146267 -0.51)
+			(start -0.146267 0.51)
+			(end 0.146267 0.51)
 			(stroke
 				(width 0.12)
@@
 		)
 		(fp_line
-			(start -0.146267 0.51)
-			(end 0.146267 0.51)
+			(start -0.146267 -0.51)
+			(end 0.146267 -0.51)
 			(stroke
 				(width 0.12)
@@
 		)
 		(fp_line
-			(start -1.65 -0.73)
-			(end 1.65 -0.73)
+			(start -1.65 0.73)
+			(end -1.65 -0.73)
 			(stroke
 				(width 0.05)
@@
 		)
 		(fp_line
-			(start -1.65 0.73)
-			(end -1.65 -0.73)
+			(start 1.65 0.73)
+			(end -1.65 0.73)
 			(stroke
 				(width 0.05)
@@
 		)
 		(fp_line
-			(start 1.65 -0.73)
-			(end 1.65 0.73)
+			(start -1.65 -0.73)
+			(end 1.65 -0.73)
 			(stroke
 				(width 0.05)
@@
 		)
 		(fp_line
-			(start 1.65 0.73)
-			(end -1.65 0.73)
+			(start 1.65 -0.73)
+			(end 1.65 0.73)
 			(stroke
 				(width 0.05)
@@
 		)
 		(fp_line
-			(start -0.8 -0.4)
-			(end 0.8 -0.4)
+			(start -0.8 0.4)
+			(end -0.8 -0.4)
 			(stroke
 				(width 0.1)
@@
 		)
 		(fp_line
-			(start -0.8 0.4)
-			(end -0.8 -0.4)
+			(start 0.8 0.4)
+			(end -0.8 0.4)
 			(stroke
 				(width 0.1)
@@
 		)
 		(fp_line
-			(start 0.8 -0.4)
-			(end 0.8 0.4)
+			(start -0.8 -0.4)
+			(end 0.8 -0.4)
 			(stroke
 				(width 0.1)
@@
 		)
 		(fp_line
-			(start 0.8 0.4)
-			(end -0.8 0.4)
+			(start 0.8 -0.4)
+			(end 0.8 0.4)
 			(stroke
 				(width 0.1)
@@
 		)
 		(fp_text user "${REFERENCE}"
-			(at 0 0 0)
+			(at 0 0 90)
 			(layer "F.Fab")
 			(effects
@@
 		)
 		(pad "1" smd roundrect
-			(at -0.8625 0)
+			(at -0.8625 0 270)
 			(size 1.075 0.95)
 			(layers "F.Cu" "F.Mask" "F.Paste")
@@
 		)
 		(pad "2" smd roundrect
-			(at 0.8625 0)
+			(at 0.8625 0 270)
 			(size 1.075 0.95)
 			(layers "F.Cu" "F.Mask" "F.Paste")
@@
 		)
 	)
-	(gr_rect
-		(start 114.71 131.54)
-		(end 139.54 136.24)
-		(stroke
-			(width 0.2)
-			(type default)
-		)
-		(fill no)
-		(layer "F.Cu")
-	)
 	(gr_line
 		(start 116.735 75.865)
@@
 		)
 	)
-	(gr_text_box "diagonal bus I sense and H bridge to 3v3, figuring out orientation\n"
-		(start 217.53 108.26)
-		(end 250.22 121.04)
-		(margins 1.0025 1.0025 1.0025 1.0025)
-		(layer "F.Cu")
-		(effects
-			(font
-				(size 1.5 1.5)
-				(thickness 0.3)
-				(bold yes)
-			)
-			(justify left top)
-		)
-		(border yes)
-		(stroke
-			(width 0.2)
-			(type solid)
-		)
-	)
 	(segment
 		(start 148.672277 120.764723)
@@
 	)
 	(via
+		(at 119.7 111.9)
+		(size 0.6)
+		(drill 0.3)
+		(layers "F.Cu" "B.Cu")
+		(free yes)
+		(net 3)
+	)
+	(via
 		(at 156.475 114.205)
 		(size 0.6)
@@
 	)
 	(via
+		(at 119.13 112.52)
+		(size 0.6)
+		(drill 0.3)
+		(layers "F.Cu" "B.Cu")
+		(free yes)
+		(net 3)
+	)
+	(via
 		(at 157.640277 113.21)
 		(size 0.6)
@@
 	)
 	(via
+		(at 119.74 111.23)
+		(size 0.6)
+		(drill 0.3)
+		(layers "F.Cu" "B.Cu")
+		(free yes)
+		(net 3)
+	)
+	(via
 		(at 143.440277 113.16)
 		(size 0.6)
@@
 	)
 	(via
+		(at 118.97 111.89)
+		(size 0.6)
+		(drill 0.3)
+		(layers "F.Cu" "B.Cu")
+		(free yes)
+		(net 3)
+	)
+	(via
 		(at 157.665277 114.205)
 		(size 0.6)
@@
 	)
 	(via
+		(at 120.54 110.46)
+		(size 0.6)
+		(drill 0.3)
+		(layers "F.Cu" "B.Cu")
+		(free yes)
+		(net 3)
+	)
+	(via
+		(at 120.46 111.21)
+		(size 0.6)
+		(drill 0.3)
+		(layers "F.Cu" "B.Cu")
+		(free yes)
+		(net 3)
+	)
+	(via
 		(at 155.925 114.705)
 		(size 0.6)
@@
 		(net 3)
 	)
+	(via
+		(at 118.45 112.46)
+		(size 0.6)
+		(drill 0.3)
+		(layers "F.Cu" "B.Cu")
+		(free yes)
+		(net 3)
+	)
 	(segment
 		(start 146.425277 117.16)
@@
 		(size 0.6)
 		(drill 0.3)
+		(layers "F.Cu" "B.Cu")
+		(net 6)
+	)
+	(via
+		(at 172.17 79.3)
+		(size 0.6)
+		(drill 0.3)

Commit message: glitching out, some stitching
Routing:
- net GNDPWR: vias 57 -> 196
- net /Control/V_{sc,+}: vias 3 -> 5

Commit message: Trevor is a genius, flipped mspm0 pins, in progress: 3v3 rerouting/redesign, edge pathing, deleting old stuff, etc.
Parts:
- removed C_{byp}1: 0.1u, Capacitor_SMD:C_0603_1608Metric_Pad1.08x0.95mm_HandSolder
- removed C_{l}1: 1n, Capacitor_SMD:C_0603_1608Metric_Pad1.08x0.95mm_HandSolder
- removed R_{pu}1: 100, Resistor_SMD:R_0603_1608Metric_Pad0.98x0.95mm_HandSolder
- removed U3: ACS71240KEXBLT-050U5, Sensor_Current:Allegro_QFN-12-10-1EP_3x3mm_P0.5mm
- moved GNDPWR2 87.2 mm to (38.9, 116.3)
- moved J3-J1 51.1 mm to (115.7, 135.1), turned to -90 degrees
- moved J4 47.4 mm to (170.1, 130.3)
- moved J2-J1 46.6 mm to (115.7, 91.9), turned to -90 degrees
- moved U4 40.8 mm to (166.6, 127.9), turned to 90 degrees
- moved GNDPWR1 9.51 mm to (108.6, 75.3)
- moved V_{sw}1 1.64 mm to (181.4, 99.1)
- moved LO_{DRV}1 1.47 mm to (184.1, 99.1)
- moved J3 1.41 mm to (176.6, 113.6)
- moved HI_{DRV}1 1.29 mm to (186.7, 99.1)
Connections:
- J1 pad 1: /Control/I_{L,out+} -> /Control/V_{sc,+}
- J1 pad 2: /Control/I_{L,out+} -> /Control/V_{sc,+}
Routing:
- net /Control/I_L: track 84.4 -> 0.00 mm, vias 3 -> 1
- net /Control/PA25: track 91.3 -> 21.6 mm, vias 3 -> 2
- net /Control/PB9: track 87.9 -> 23.7 mm, vias 2 -> 1
- net /Control/F_L: track 63.3 -> 0.00 mm, vias 3 -> 0
- net /Control/PA8: track 97.2 -> 37.8 mm, vias 3 -> 2
- net /Control/F_bat: track 63.3 -> 120.7 mm, vias 2 -> 3
- net /Control/PA22: track 92.1 -> 37.8 mm
- net /Control/I_bat: track 55.6 -> 109.2 mm
- net unconnected-(J2-J1-Pin_17-Pad17): track 0.00 -> 45.3 mm, vias 0 -> 1
- net /Control/+3V3: track 72.6 -> 116.2 mm, vias 12 -> 10
- net /Control/I_{bat,out+}: track 100.3 -> 61.6 mm, vias 31 -> 35
- net unconnected-(J2-J1-Pin_7-Pad7): track 0.00 -> 36.9 mm, vias 0 -> 1
- net unconnected-(J2-J1-Pin_18-Pad18): track 0.00 -> 36.7 mm, vias 0 -> 1
- net unconnected-(J2-J1-Pin_8-Pad8): track 0.00 -> 30.3 mm, vias 0 -> 1
- net unconnected-(J2-J1-Pin_14-Pad14): track 0.00 -> 26.8 mm, vias 0 -> 1
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- added copper zone on B.Cu, net Net-(J4-Pin_1)
- added copper zone on F.Cu, net Net-(J4-Pin_1)
- added copper zone on In1.Cu, net Net-(J4-Pin_1)
- added copper zone on In2.Cu, net Net-(J4-Pin_1)
- removed copper zone on B.Cu, net /Control/I_{L,out+}
- removed copper zone on F.Cu, net /Control/I_{L,out+}
- removed copper zone on In1.Cu, net /Control/I_{L,out+}
- removed copper zone on In2.Cu, net /Control/I_{L,out+}
Other:
- board text added: "4 pins on top only, need to route, redo 3 tp? they are: PA15 PA16 I_L/PA24 F_L/PB23? A: can remove, use pb12? WAIT FOR EGAN DO END"

Commit message: put filters closer to IC's, cleared up some stuff, still gonna have cool cross board bus prob yipee
Parts:
- C_{byp}2, C_{l}2, C_{smooth}2, R_{RC}2, R_{pu}2, R_{sens,bottom}1: moved to F.Cu
- moved C_{byp}2 48.3 mm to (166.3, 128.2), turned to 180 degrees
- moved C_{l}2 44.0 mm to (169.7, 127.4), turned to 180 degrees
- moved R_{pu}2 40.5 mm to (166.0, 126.7), turned to 0 degrees
- moved R_{RC}2 7.23 mm to (162.9, 89.5), turned to 0 degrees
- moved C_{RC}2 3.45 mm to (163.4, 88.4), turned to 0 degrees
- moved C_{RC}1 3.25 mm to (176.8, 83.1), turned to 0 degrees
- moved R_{sens,bottom}1 2.78 mm to (161.4, 91.1), turned to 0 degrees
- moved C_{smooth}2 2.11 mm to (157.9, 89.8)
- moved R_{sens,bottom}2 1.71 mm to (164.0, 90.9)
- moved J2-J1 1.08 mm to (115.5, 90.9)
- moved J3-J1 1.08 mm to (115.5, 134.1)
- moved R1 0.75 mm to (169.4, 94.8)
Routing:
- net /Control/PA15: track 74.2 -> 0.00 mm, vias 2 -> 0
- net /Control/I_{bat,out+}: track 61.6 -> 0.00 mm, vias 35 -> 34
- net /Control/F_bat: track 120.7 -> 61.8 mm, vias 3 -> 2
- net /Control/+3V3: track 116.2 -> 60.4 mm, vias 10 -> 6
- net /Control/I_bat: track 109.2 -> 56.5 mm
- net /Control/PA16: track 50.7 -> 0.00 mm, vias 2 -> 0
- net unconnected-(J2-J1-Pin_17-Pad17): track 45.3 -> 0.00 mm, vias 1 -> 0
- net unconnected-(J2-J1-Pin_7-Pad7): track 36.9 -> 0.00 mm, vias 1 -> 0
- net unconnected-(J2-J1-Pin_18-Pad18): track 36.7 -> 0.00 mm, vias 1 -> 0
- net unconnected-(J2-J1-Pin_8-Pad8): track 30.3 -> 0.00 mm, vias 1 -> 0
- net unconnected-(J2-J1-Pin_14-Pad14): track 26.8 -> 0.00 mm, vias 1 -> 0
- net unconnected-(J2-J1-Pin_13-Pad13): track 24.5 -> 0.00 mm
- net unconnected-(J2-J1-Pin_16-Pad16): track 24.5 -> 0.00 mm, vias 2 -> 0
- net /Voltage Converter/LO_DRV_{2}: track 51.4 -> 29.8 mm
- net /Control/V_{sc,+}: track 71.9 -> 50.4 mm, vias 1 -> 2
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- removed copper zone on F.Cu, net GND
- removed copper zone on In1.Cu, net GND
Other:
- board text added: "3v3 and gnd are just powering => put the outputs pa15/16 close to mspm0"
- board text added: "4 pins on top only, need to route, redo 3 tp? they are: PA15 mainly these 2 PA16 mainly these 2 I_L/PA24 these 2 gone with i sense that removed? F_L/PB23? A: can remove, use pb12? WAIT FOR EGAN DO END"
- board text removed: "4 pins on top only, need to route, redo 3 tp? they are: PA15 PA16 I_L/PA24 F_L/PB23? A: can remove, use pb12? WAIT FOR EGAN DO END"

Commit message: done, routed everything, todo: DRC
Parts:
- moved U6 149.9 mm to (99.1, 43.7)
- moved C_{RC}1 66.3 mm to (138.0, 136.9), turned to 180 degrees
- moved R_{RC}1 65.0 mm to (139.7, 136.6), turned to 0 degrees
- moved C_{RC}2 51.0 mm to (131.8, 128.4), turned to 180 degrees
- moved R_{RC}2 49.2 mm to (133.6, 129.0)
- moved HI_{DRV}2 0.74 mm to (134.6, 137.2)
- moved LO_{DRV}2 0.74 mm to (132.0, 139.1)
Routing:
- net GND: track 64.2 -> 160.2 mm, vias 8 -> 11
- net /Control/V_{sc,sens}: track 4.24 -> 96.8 mm, vias 1 -> 5
- net /Control/+3V3: track 60.4 -> 152.2 mm, vias 6 -> 7
- net /Control/F_bat: track 61.8 -> 129.7 mm
- net /Control/V_{bat,sens}: track 3.72 -> 67.8 mm, vias 1 -> 3
- net /Control/I_{bat,out+}: track 0.00 -> 59.4 mm, vias 34 -> 38
- net /Control/I_bat: track 56.5 -> 95.0 mm, vias 1 -> 2
- net /Control/PA25: track 21.6 -> 51.6 mm
- net /Control/PA22: track 37.8 -> 62.9 mm, vias 4 -> 5
- net /Control/PA8: track 37.8 -> 62.7 mm
- net /Control/PB9: track 23.7 -> 44.3 mm, vias 1 -> 2
- net /Voltage Converter/LO_DRV_{2}: track 29.8 -> 43.7 mm
- net /Voltage Converter/HI_DRV_{2}: track 17.1 -> 28.9 mm
- net /Control/PA15: track 0.00 -> 6.19 mm
- net /Control/V_{sc,+}: track 50.4 -> 53.8 mm
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
Commit message: DRC, cleared up all errors except 2 that are unavoidable with board settings (2 pads on the same ic being too close). Warnings are vast majority of the silkscreen, solder mask type. A few important warnings to check: footprint does not match library, from modifying them, reassigning pins, etc. should double check those.
Parts:
- moved C_{bulk,out}1 0.15 mm to (156.0, 120.8)
- moved C_{d1}1 0.05 mm to (163.5, 121.1)
- moved C_{d2}1 0.05 mm to (160.2, 121.1)
- moved C_{d6}1 0.05 mm to (156.9, 121.1)
Routing:
- net /Control/F_bat: track 129.7 -> 96.2 mm
- net GNDPWR: track 3.97 -> 0.00 mm
- net /Control/PA22: track 62.9 -> 66.4 mm, vias 5 -> 4
- net /Voltage Converter/HI_DRV_{2}: track 28.9 -> 26.3 mm, vias 1 -> 0
- net /Housekeeping/+12V: track 30.6 -> 32.0 mm
- net /Control/PA8: track 62.7 -> 64.0 mm, vias 2 -> 1
- net /Control/V_{sc,+}: track 53.8 -> 53.1 mm
- net /Voltage Converter/V_{sw,2}: track 63.1 -> 63.5 mm, vias 10 -> 11
- net /Control/V_{sc,sens}: vias 5 -> 4

Commit message: small
Parts:
- moved U6 98.9 mm to (198.0, 41.0)
Other:
- board text added: "UT Robomasters Electrical Subteam Egan Wang Trevor White Daniel Zhou"
- board text removed: "3v3 and gnd are just powering => put the outputs pa15/16 close to mspm0"
- board text removed: "4 pins on top only, need to route, redo 3 tp? they are: PA15 mainly these 2 PA16 mainly these 2 I_L/PA24 these 2 gone with i sense that removed? F_L/PB23? A: can remove, use pb12? WAIT FOR EGAN DO END"
- board text removed: "UT Robomasters Electrical Subteam"
Changed lines of the file:
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@@
 	(footprint "MSPM0:ti_LP_MSPM0G3507"
 		(layer "F.Cu")
-		(at 99.1 43.67 -90)
+		(at 197.99 40.98 -90)
 		(property "Reference" "U6"
 			(at -22.86 -45.72 90)
@@
 			(layer "Cmts.User")
 			(pts
-				(xy 101.64 51.29) (xy 152.44 51.29)
+				(xy 200.53 48.6) (xy 251.33 48.6)
 			)
 			(height 5.08)
@@
 			)
 			(gr_text "2.000"
-				(at 127.04 55.27 0)
+				(at 225.93 52.58 0)
 				(layer "Cmts.User")
 				(effects
@@
 			(layer "Cmts.User")
 			(pts
-				(xy 132.12 15.73) (xy 132.12 71.61)
+				(xy 231.01 13.04) (xy 231.01 68.92)
 			)
 			(height -2.54)
@@
 			)
 			(gr_text "2.200"
-				(at 133.56 43.67 90)
+				(at 232.45 40.98 90)
 				(layer "Cmts.User")
 				(effects
@@
 			(layer "Cmts.User")
 			(pts
-				(xy 78.78 56.37) (xy 48.3 56.37)
+				(xy 177.67 53.68) (xy 147.19 53.68)
 			)
 			(height -2.54)
@@
 			)
 			(gr_text "1.200"
-				(at 63.54 57.81 0)
+				(at 162.43 55.12 0)
 				(layer "Cmts.User")
 				(effects
@@
 			(layer "Cmts.User")
 			(pts
-				(xy 152.44 30.97) (xy 48.3 30.97)
+				(xy 251.33 28.28) (xy 147.19 28.28)
 			)
 			(height -5.08)
@@
 			)
 			(gr_text "4.100"
-				(at 100.37 34.95 0)
+				(at 199.26 32.26 0)
 				(layer "Cmts.User")
 				(effects
@@
 		(layer "Edge.Cuts")
 	)
-	(gr_text "3v3 and gnd are just powering\n=> put the outputs pa15/16 close to mspm0"
-		(at 144.49 65.17 -0)
-		(layer "F.Cu")
-		(effects
-			(font
-				(size 1.5 1.5)
-				(thickness 0.3)
-				(bold yes)
-			)
-			(justify left bottom)
-		)
-	)
-	(gr_text "4 pins on top only, need to route, redo 3 tp?\nthey are:\nPA15	mainly these 2\nPA16	mainly these 2\n\nI_L/PA24	these 2 gone with i sense that removed?\nF_L/PB23? A: can remove, use pb12?\nWAIT FOR EGAN DO END"
-		(at 211.67 112.72 0)
-		(layer "F.Cu")
-		(effects
-			(font
-				(size 1.5 1.5)
-				(thickness 0.3)
-				(bold yes)
-			)
-			(justify left bottom)
-		)
-	)
-	(gr_text "UT Robomasters\nElectrical Subteam"
-		(at 87.05 31.17 0)
+	(gr_text "UT Robomasters\nElectrical Subteam\nEgan Wang\nTrevor White\nDaniel Zhou"
+		(at 98.61 92.21 0)
 		(layer "F.SilkS")
 		(effects
@@
 	)
 	(gr_text "Supercap\nBoard"
-		(at 87.7 27.82 0)
+		(at 99.18 84.13 0)
 		(layer "F.SilkS")
 		(effects

Commit message: starting on V3 :) yipee. finished pours and stuff
Parts:
- moved P7803B-1000R1 45.5 mm to (183.3, 120.2)
- moved V_{MiniPC}1 45.5 mm to (180.4, 131.3)
- moved C_{smooth}3 43.2 mm to (171.0, 123.4)
- moved R4 43.2 mm to (173.2, 128.3)
- moved U1 43.2 mm to (172.8, 121.8)
- moved C_{smooth}1 43.2 mm to (176.4, 120.5)
- moved R3 43.2 mm to (172.3, 126.6)
- moved C_{smooth}2 39.7 mm to (159.4, 129.5), turned to 90 degrees
- moved U2 36.3 mm to (161.3, 127.9), turned to -90 degrees
- moved R_{sens,bottom}1 34.9 mm to (160.8, 126.0), turned to 90 degrees
- moved LO_{DRV}1 34.4 mm to (157.8, 121.3)
- moved V_{sw}1 34.4 mm to (155.2, 121.4)
- moved HI_{DRV}1 34.4 mm to (160.5, 121.3)
- moved R_{sens,bottom}2 32.7 mm to (160.5, 123.4), turned to 180 degrees
- moved J2 25.9 mm to (153.5, 106.9)
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Routing:
- net /Control/+3V3: track 152.2 -> 42.9 mm, vias 7 -> 6
- net GND: track 160.1 -> 66.4 mm, vias 11 -> 10
- net /Control/V_{sc,sens}: track 96.8 -> 4.24 mm, vias 4 -> 1
- net /Control/F_bat: track 96.2 -> 25.3 mm
- net /Control/I_bat: track 95.0 -> 28.0 mm, vias 2 -> 1
- net /Control/V_{bat,sens}: track 67.8 -> 2.09 mm, vias 3 -> 1
- net /Control/I_{bat,out+}: track 59.6 -> 0.00 mm, vias 38 -> 34
- net /Voltage Converter/V_{sw,2}: track 63.5 -> 7.37 mm, vias 11 -> 9
- net /Control/V_{sc,+}: track 53.1 -> 2.00 mm, vias 2 -> 0
- net /Voltage Converter/V_{sw,1}: track 76.3 -> 25.7 mm
- net /Voltage Converter/HI_DRV_{1}: track 68.8 -> 23.1 mm
- net /Voltage Converter/LO_DRV_{1}: track 74.1 -> 36.0 mm
- net /Control/PA25: track 51.6 -> 80.3 mm
- net /Control/PB9: track 44.3 -> 72.6 mm
- net /Control/PA8: track 64.0 -> 92.1 mm
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