File: Supercap.kicad_sch (KiCad schematic)
At the start: 3 parts

Commit message: big progress on layout
Connections:
- net Control/I_{out sense-} is gone; now on net Control/I_{bat,out+}: V_{out}1.2 (Pin_2)
Other:
- sheet Control ports: added none; removed I_{out sense+}, I_{out sense-}
Changed lines of the file:
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@@
-	(wire
-		(pts
-			(xy 133.35 66.04) (xy 208.28 66.04)
-		)
-		(stroke
-			(width 0)
-			(type default)
-		)
-	)
 	(wire
 		(pts
@@
 		)
 	)
-	(wire
-		(pts
-			(xy 135.89 77.47) (xy 135.89 68.58)
-		)
-		(stroke
-			(width 0)
-			(type default)
-		)
-	)
 	(polyline
 		(pts
@@
 		)
 	)
-	(wire
-		(pts
-			(xy 212.09 68.58) (xy 212.09 60.96)
-		)
-		(stroke
-			(width 0)
-			(type default)
-		)
-	)
 	(polyline
 		(pts
@@
 	(wire
 		(pts
-			(xy 135.89 68.58) (xy 212.09 68.58)
-		)
-		(stroke
-			(width 0)
-			(type default)
-		)
-	)
-	(wire
-		(pts
 			(xy 198.12 97.79) (xy 205.74 97.79)
 		)
@@
 		)
 	)
-	(wire
-		(pts
-			(xy 133.35 77.47) (xy 133.35 66.04)
-		)
-		(stroke
-			(width 0)
-			(type default)
-		)
-	)
 	(polyline
 		(pts
@@
 		)
 	)
-	(wire
-		(pts
-			(xy 208.28 66.04) (xy 208.28 60.96)
-		)
-		(stroke
-			(width 0)
-			(type default)
-		)
-	)
 	(polyline
 		(pts
@@
 	(wire
 		(pts
-			(xy 212.09 60.96) (xy 232.41 60.96)
-		)
-		(stroke
-			(width 0)
-			(type default)
-		)
-	)
-	(wire
-		(pts
 			(xy 148.59 111.76) (xy 205.74 111.76)
 		)
@@
 	(wire
 		(pts
-			(xy 177.8 60.96) (xy 208.28 60.96)
+			(xy 177.8 60.96) (xy 232.41 60.96)
 		)
 		(stroke
@@
 			(effects
 				(font
-					(size 1.27 1.27)
-				)
-				(justify right)
-			)
-		)
-		(pin "I_{out sense+}" bidirectional
-			(at 133.35 77.47 90)
-			(effects
-				(font
-					(size 1.27 1.27)
-				)
-				(justify right)
-			)
-		)
-		(pin "I_{out sense-}" bidirectional
-			(at 135.89 77.47 90)
-			(effects
-				(font

Commit message: Trevor is a genius, flipped mspm0 pins, in progress: 3v3 rerouting/redesign, edge pathing, deleting old stuff, etc.
Other:
- sheet Control ports: added none; removed I_{L,out+}
Changed lines of the file:
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@@
+	)
+	(junction
+		(at 201.93 82.55)
+		(diameter 0)
+		(color 0 0 0 0)
 	)
 	(junction
@@
 	(wire
 		(pts
+			(xy 152.4 97.79) (xy 152.4 107.95)
+		)
+		(stroke
+			(width 0)
+			(type default)
+		)
+	)
+	(wire
+		(pts
 			(xy 102.87 92.71) (xy 100.33 92.71)
 		)
@@
 	(wire
 		(pts
-			(xy 153.67 106.68) (xy 153.67 95.25)
-		)
-		(stroke
-			(width 0)
-			(type default)
-		)
-	)
-	(wire
-		(pts
 			(xy 148.59 100.33) (xy 148.59 111.76)
 		)
@@
 	(wire
 		(pts
-			(xy 144.78 97.79) (xy 151.13 97.79)
-		)
-		(stroke
-			(width 0)
-			(type default)
-		)
-	)
-	(wire
-		(pts
 			(xy 92.71 82.55) (xy 102.87 82.55)
 		)
@@
 	(wire
 		(pts
+			(xy 198.12 82.55) (xy 201.93 82.55)
+		)
+		(stroke
+			(width 0)
+			(type default)
+		)
+	)
+	(wire
+		(pts
 			(xy 177.8 60.96) (xy 177.8 77.47)
 		)
@@
 		)
 	)
-	(wire
-		(pts
-			(xy 151.13 109.22) (xy 203.2 109.22)
-		)
-		(stroke
-			(width 0)
-			(type default)
-		)
-	)
 	(polyline
 		(pts
@@
 		)
 	)
+	(wire
+		(pts
+			(xy 201.93 107.95) (xy 201.93 82.55)
+		)
+		(stroke
+			(width 0)
+			(type default)
+		)
+	)
 	(polyline
 		(pts
@@
 		)
 	)
+	(wire
+		(pts
+			(xy 144.78 97.79) (xy 152.4 97.79)
+		)
+		(stroke
+			(width 0)
+			(type default)
+		)
+	)
 	(polyline
 		(pts
@@
 		)
 	)
-	(wire
-		(pts
-			(xy 153.67 95.25) (xy 144.78 95.25)
-		)
-		(stroke
-			(width 0)
-			(type default)
-		)
-	)
 	(polyline
 		(pts
@@
 	(wire
 		(pts
-			(xy 151.13 97.79) (xy 151.13 109.22)
-		)
-		(stroke
-			(width 0)
-			(type default)
-		)
-	)
-	(wire
-		(pts
 			(xy 67.31 60.96) (xy 97.79 60.96)
 		)
@@
 		)
 	)
-	(wire
-		(pts
-			(xy 198.12 82.55) (xy 200.66 82.55)
-		)
-		(stroke
-			(width 0)
-			(type default)
-		)
-	)
 	(polyline
 		(pts
@@
 		)
 	)
-	(wire
-		(pts
-			(xy 200.66 106.68) (xy 153.67 106.68)
-		)
-		(stroke
-			(width 0)
-			(type default)
-		)
-	)
-	(wire
-		(pts
-			(xy 203.2 109.22) (xy 203.2 82.55)
-		)
-		(stroke
-			(width 0)
-			(type default)
-		)
-	)
 	(polyline
 		(pts
@@
 		)
 	)
+	(wire
+		(pts
+			(xy 201.93 82.55) (xy 208.28 82.55)
+		)
+		(stroke
+			(width 0)
+			(type default)
+		)
+	)
 	(polyline
 		(pts
@@
 	(wire
 		(pts
-			(xy 203.2 82.55) (xy 208.28 82.55)
+			(xy 152.4 107.95) (xy 201.93 107.95)
 		)
 		(stroke
@@
 			(width 0.635)
 			(type solid)
-		)
-	)
-	(wire
-		(pts
-			(xy 200.66 82.55) (xy 200.66 106.68)
-		)
-		(stroke
-			(width 0)
-			(type default)
 		)
 	)
@@
 			)
 		)
-		(pin "I_{L,out+}" bidirectional
-			(at 144.78 95.25 0)
-			(effects
-				(font
-					(size 1.27 1.27)
-				)
-				(justify right)
-			)
-		)

Commit message: split into separate boards as per regulations
Parts:
- added V_{sc}1: Conn_01x02_Pin, Connector_AMASS:AMASS_XT30PW-M_1x02_P2.50mm_Horizontal, symbol Connector:Conn_01x02_Pin
- V_{in}1: footprint Connector_AMASS:AMASS_XT30PW-F_1x02_P2.50mm_Horizontal -> Connector_AMASS:AMASS_XT30PW-M_1x02_P2.50mm_Horizontal
Connections:
- net Control/V_{sc,+}: now also V_{sc}1.2 (Pin_2)
- net Control/V_{sc,-}: now also V_{sc}1.1 (Pin_1)
Other:
- removed sheet Supercap Board
- note added: "12V Gate Driver 3V3 Signals"
- note removed: "4P Capacitors"
Changed lines of the file:
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@@
-		)
-	)
-	(rectangle
-		(start 215.9 81.28)
-		(end 233.68 99.06)
-		(stroke
-			(width 0)
-			(type default)
-		)
-		(fill
-			(type none)
 		)
 	)
@@
 		)
 	)
-	(text "4P\nCapacitors"
+	(text "12V Gate Driver\n3V3 Signals"
 		(exclude_from_sim no)
-		(at 241.3 89.916 0)
+		(at 72.136 90.043 0)
 		(effects
 			(font
-				(size 1.27 1.27)
+				(size 1.905 1.905)
 			)
 		)
@@
 	)
 	(junction
-		(at 205.74 97.79)
-		(diameter 0)
-		(color 0 0 0 0)
-	)
-	(junction
 		(at 177.8 60.96)
 		(diameter 0)
 		(color 0 0 0 0)
 	)
-	(polyline
-		(pts
-			(xy 224.79 91.44) (xy 224.79 95.25)
-		)
-		(stroke
-			(width 0)
-			(type default)
-		)
+	(junction
+		(at 205.74 85.09)
+		(diameter 0)
+		(color 0 0 0 0)
 	)
 	(polyline
@@
 		)
 	)
-	(polyline
-		(pts
-			(xy 218.44 91.44) (xy 231.14 91.44)
-		)
-		(stroke
-			(width 0)
-			(type default)
-		)
-	)
 	(wire
 		(pts
@@
 		)
 	)
+	(wire
+		(pts
+			(xy 201.93 82.55) (xy 201.93 107.95)
+		)
+		(stroke
+			(width 0)
+			(type default)
+		)
+	)
 	(polyline
 		(pts
@@
 	(polyline
 		(pts
-			(xy 218.44 88.9) (xy 231.14 88.9)
-		)
-		(stroke
-			(width 0)
-			(type default)
-		)
-	)
-	(polyline
-		(pts
 			(xy 115.57 90.17) (xy 118.11 90.17)
 		)
@@
 		)
 	)
-	(wire
-		(pts
-			(xy 201.93 107.95) (xy 201.93 82.55)
-		)
-		(stroke
-			(width 0)
-			(type default)
-		)
-	)
 	(polyline
 		(pts
@@
 		)
 	)
-	(polyline
-		(pts
-			(xy 224.79 85.09) (xy 224.79 88.9)
+	(wire
+		(pts
+			(xy 201.93 82.55) (xy 210.82 82.55)
 		)
 		(stroke
@@
 	(wire
 		(pts
-			(xy 198.12 97.79) (xy 205.74 97.79)
+			(xy 198.12 85.09) (xy 205.74 85.09)
 		)
 		(stroke
@@
 	(wire
 		(pts
-			(xy 205.74 97.79) (xy 205.74 111.76)
+			(xy 205.74 85.09) (xy 205.74 111.76)
 		)
 		(stroke
@@
 		)
 	)
-	(wire
-		(pts
-			(xy 201.93 82.55) (xy 208.28 82.55)
-		)
-		(stroke
-			(width 0)
-			(type default)
-		)
-	)
 	(polyline
 		(pts
@@
 	(wire
 		(pts
-			(xy 205.74 97.79) (xy 208.28 97.79)
+			(xy 205.74 85.09) (xy 210.82 85.09)
 		)
 		(stroke
@@
 			)
 		)
-		(property "Footprint" "Connector_AMASS:AMASS_XT30PW-F_1x02_P2.50mm_Horizontal"
+		(property "Footprint" "Connector_AMASS:AMASS_XT30PW-M_1x02_P2.50mm_Horizontal"
 			(at 54.61 63.5 0)
 			(effects
@@
 				(path "/98ee8313-37ab-4329-91ab-b5710476f82f"
 					(reference "V_{in}1")
+					(unit 1)
+				)
+			)
+		)
+	)
+	(symbol
+		(lib_id "Connector:Conn_01x02_Pin")
+		(at 215.9 85.09 180)
+		(unit 1)
+		(exclude_from_sim no)
+		(in_bom no)
+		(on_board yes)
+		(dnp no)
+		(property "Reference" "V_{sc}1"
+			(at 224.155 85.344 0)
+			(effects
+				(font
+					(size 1.27 1.27)
+				)
+			)
+		)
+		(property "Value" "Conn_01x02_Pin"
+			(at 224.155 82.804 0)
+			(effects
+				(font
+					(size 1.27 1.27)
+				)
+			)
+		)
+		(property "Footprint" "Connector_AMASS:AMASS_XT30PW-M_1x02_P2.50mm_Horizontal"
+			(at 215.9 85.09 0)
+			(effects
+				(font
+					(size 1.27 1.27)
+				)
+				(hide yes)
+			)
+		)
+		(property "Datasheet" ""
+			(at 215.9 85.09 0)
+			(effects
+				(font
+					(size 1.27 1.27)
+				)
+				(hide yes)
+			)
+		)
+		(property "Description" "Generic connector, single row, 01x02, script generated"
+			(at 215.9 85.09 0)
+			(effects
+				(font
+					(size 1.27 1.27)
+				)
+				(hide yes)
+			)
+		)
+		(property "Digi-Key Part Number" ""
+			(at 215.9 85.09 0)
+			(effects
+				(font
+					(size 1.27 1.27)
+				)
+				(hide yes)
+			)
+		)
+		(pin "2"
+		)
+		(pin "1"
+		)
+		(instances
+			(project "Supercap"
+				(path "/98ee8313-37ab-4329-91ab-b5710476f82f"
+					(reference "V_{sc}1")
 					(unit 1)
 				)
@@
 		)
 		(pin "V_{cap-}" bidirectional
-			(at 198.12 97.79 0)
+			(at 198.12 85.09 0)
 			(effects
 				(font
@@
 				)
 			)
-		)
-	)
-	(sheet
-		(at 208.28 77.47)
-		(size 41.91 25.4)
-		(exclude_from_sim no)
-		(in_bom yes)
-		(on_board yes)
-		(dnp no)
-		(fields_autoplaced yes)
-		(stroke
-			(width 0.1524)
-			(type solid)
-		)
-		(fill
-			(color 0 0 0 0.0000)
-		)
-		(property "Sheetname" "Supercap Board"
-			(at 208.28 76.7584 0)
-			(effects
-				(font
-					(size 1.27 1.27)
-				)
-				(justify left bottom)
-			)
-		)
-		(property "Sheetfile" "Supercap_Board/supercap_board.kicad_sch"
-			(at 208.28 103.4546 0)
-			(effects
-				(font
-					(size 1.27 1.27)
-				)
-				(justify left top)
-			)
-		)
-		(pin "V_{cap+}" bidirectional
-			(at 208.28 82.55 180)
-			(effects
-				(font
-					(size 1.27 1.27)
-				)
-				(justify left)
-			)
-		)
-		(pin "V_{cap-}" bidirectional
-			(at 208.28 97.79 180)
-			(effects
-				(font
-					(size 1.27 1.27)
-				)
-				(justify left)
-			)
-		)
-		(instances
-			(project "Supercap"
-				(path "/98ee8313-37ab-4329-91ab-b5710476f82f"
-					(page "5")
-				)
-			)

Commit message: cleaned up PCB after meeting with BBJ
Parts:
- V_{MiniPC}1, V_{out}1: footprint Connector_AMASS:AMASS_XT30PW-F_1x02_P2.50mm_Horizontal -> Robomaster_Conn:AMASS_XT30PW-F_1x02_P2.50mm_Horizontal
- V_{in}1, V_{sc}1: footprint Connector_AMASS:AMASS_XT30PW-M_1x02_P2.50mm_Horizontal -> Robomaster_Conn:AMASS_XT30PW-M_1x02_P2.50mm_Horizontal
Changed lines of the file:
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@@
 			)
 		)
-		(property "Footprint" "Connector_AMASS:AMASS_XT30PW-F_1x02_P2.50mm_Horizontal"
+		(property "Footprint" "Robomaster_Conn:AMASS_XT30PW-F_1x02_P2.50mm_Horizontal"
 			(at 38.1 82.55 0)
 			(effects
@@
 			)
 		)
-		(property "Footprint" "Connector_AMASS:AMASS_XT30PW-M_1x02_P2.50mm_Horizontal"
+		(property "Footprint" "Robomaster_Conn:AMASS_XT30PW-M_1x02_P2.50mm_Horizontal"
 			(at 54.61 63.5 0)
 			(effects
@@
 			)
 		)
-		(property "Footprint" "Connector_AMASS:AMASS_XT30PW-M_1x02_P2.50mm_Horizontal"
+		(property "Footprint" "Robomaster_Conn:AMASS_XT30PW-M_1x02_P2.50mm_Horizontal"
 			(at 215.9 85.09 0)
 			(effects
@@
 			)
 		)
-		(property "Footprint" "Connector_AMASS:AMASS_XT30PW-F_1x02_P2.50mm_Horizontal"
+		(property "Footprint" "Robomaster_Conn:AMASS_XT30PW-F_1x02_P2.50mm_Horizontal"
 			(at 237.49 63.5 0)
 			(effects
